File: Hardware/Haar.sch (EAGLE design)
At the start: 15 parts, among them J1 CONN_42.54, Q1 2N7002, U1 SHT35DFN, U2 LPS35HW, U4 TPS62237DRY, U5 TXS0102DQM

Commit message: Fixed ISP error, updated notes
Fixed an errant connection to the ISP header on both versions in schematic, still need to fix the layout. Also removed outdated notes on schematic
Connections:
- net SCL: no longer ISP1.MOSI
- net SDA_EXT: now also ISP1.MOSI
Other:
- note removed: "Add BUCK_MODE!"
- note removed: "Connect RH_INT and RH_RST lines!"
Changed lines of the file:
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@@
 <sheet>
 <plain>
-<text x="55.88" y="63.5" size="1.778" layer="91">MOSI</text>
+<text x="58.42" y="86.36" size="1.778" layer="91">MOSI</text>
 <text x="55.88" y="83.82" size="1.778" layer="91">MISO</text>
 <text x="58.42" y="73.66" size="1.778" layer="91">SCK</text>
 <text x="58.42" y="71.12" size="1.778" layer="91">INT0</text>
-<text x="22.86" y="48.26" size="1.778" layer="91">Connect RH_INT
-and RH_RST lines!</text>
-<text x="96.52" y="63.5" size="1.778" layer="91">Add BUCK_MODE!</text>
 </plain>
 <instances>
@@
 <label x="78.74" y="109.22" size="1.778" layer="95"/>
 </segment>
+<segment>
+<pinref part="ISP1" gate="G$1" pin="MOSI"/>
+<wire x1="40.64" y1="129.54" x2="45.72" y2="129.54" width="0.1524" layer="91"/>
+<label x="43.18" y="129.54" size="1.778" layer="95"/>
+</segment>
 </net>
 <net name="RX" class="0">
@@
 <wire x1="109.22" y1="22.86" x2="114.3" y2="22.86" width="0.1524" layer="91"/>
 <label x="111.76" y="22.86" size="1.778" layer="95"/>
-</segment>
-<segment>
-<pinref part="ISP1" gate="G$1" pin="MOSI"/>
-<wire x1="40.64" y1="129.54" x2="45.72" y2="129.54" width="0.1524" layer="91"/>
-<label x="43.18" y="129.54" size="1.778" layer="95"/>
 </segment>
 </net>
@@
 </drawing>
 <compatibility>
-<note version="6.3" minversion="6.2.2" severity="warning">
-Since Version 6.2.2 text objects can contain more than one line,
-which will not be processed correctly with this version.
-</note>
 <note version="8.2" severity="warning">
 Since Version 8.2, EAGLE supports online libraries. The ids
