File: Hardware/Haar_HardMount.brd (EAGLE design)
At the start: 30.4 x 10.1 mm, 15 parts, among them J1 SOLDERCUP_CONN_QUAD, Q1 2N7002, U1 SHT35DFN, U2 LPS35HW, U4 TPS62237DRY, U5 TXS0102DQM

Commit message: Minor cleanup on board, fixed #1, sent v0.1 to fab
Minor board cleanup, added pullup resistors on internal I2C lines, fixed #1 issue
Parts:
- added R2, R3: (no value), bschulz_passives:R0402
- moved ISP1 0.13 mm to (13.0, 7.37)
- moved C4 0.13 mm to (16.6, 7.62)
Connections:
- net 3V3: now also R2.2, R3.2
- net SCL: now also R2.1
- net SDA: now also R3.1
Routing:
- net SCL: track 15.0 -> 22.8 mm, vias 3 -> 4
- net 3V3: track 57.4 -> 59.7 mm
- net SDA: track 17.4 -> 18.2 mm
Other:
- board text added: "Project Haar v0.1 ---------------- Developed by Northern Widget and University of Minnesota"
- board text added: "SCL"
- board text added: "SDA"
- board text added: "Vin+"
- board text added: "Vin-"
- board text removed: "Project Haar v0.0 ---------------- Developed by Northern Widget and University of Minnesota"

Commit message: Generated fab quote
Updated part values for inductor and capacitor in Eagle, generated new BoM and zipped into file for quote generation
Parts:
- R2, R3: value (none) -> 10k
Changed lines of the file:
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@@
 <?xml version="1.0" encoding="utf-8"?>
 <!DOCTYPE eagle SYSTEM "eagle.dtd">
-<eagle version="9.4.2">
+<eagle version="9.5.2">
 <drawing>
 <settings>
-<setting alwaysvectorfont="yes"/>
+<setting alwaysvectorfont="no"/>
 <setting verticaltext="up"/>
 </settings>
@@
 <elements>
 <element name="C1" library="bschulz_passives" package="C0402" value="4.7uF" x="5.207" y="7.112" smashed="yes" rot="R270">
-<attribute name="DIGIKEY" value="" x="-15.113" y="-8.128" size="1.778" layer="27" rot="R270" display="off"/>
-<attribute name="MF" value="" x="-15.113" y="-8.128" size="1.778" layer="27" rot="R270" display="off"/>
-<attribute name="MPN" value="" x="-15.113" y="-8.128" size="1.778" layer="27" rot="R270" display="off"/>
+<attribute name="DIGIKEY" value="490-14306-1-ND" x="-15.113" y="-8.128" size="1.778" layer="27" rot="R270" display="off"/>
+<attribute name="MF" value="Murata" x="-15.113" y="-8.128" size="1.778" layer="27" rot="R270" display="off"/>
+<attribute name="MPN" value="GRM155R61A475MEAAD" x="-15.113" y="-8.128" size="1.778" layer="27" rot="R270" display="off"/>
 <attribute name="NAME" x="4.318" y="7.366" size="0.6096" layer="25" font="vector" ratio="15" rot="R270" align="center"/>
 <attribute name="VALUE" x="3.81" y="7.112" size="0.6096" layer="27" font="vector" ratio="15" rot="R270" align="center"/>
 </element>
 <element name="C2" library="bschulz_passives" package="C0402" value="4.7uF" x="7.239" y="5.334" smashed="yes" rot="R180">
-<attribute name="DIGIKEY" value="" x="-13.081" y="25.654" size="1.778" layer="27" rot="R180" display="off"/>
-<attribute name="MF" value="" x="-13.081" y="25.654" size="1.778" layer="27" rot="R180" display="off"/>
-<attribute name="MPN" value="" x="-13.081" y="25.654" size="1.778" layer="27" rot="R180" display="off"/>
+<attribute name="DIGIKEY" value="490-14306-1-ND" x="-13.081" y="25.654" size="1.778" layer="27" rot="R180" display="off"/>
+<attribute name="MF" value="Murata" x="-13.081" y="25.654" size="1.778" layer="27" rot="R180" display="off"/>
+<attribute name="MPN" value="GRM155R61A475MEAAD" x="-13.081" y="25.654" size="1.778" layer="27" rot="R180" display="off"/>
 <attribute name="NAME" x="8.128" y="4.445" size="0.6096" layer="25" font="vector" ratio="15" rot="R180" align="center"/>
 <attribute name="VALUE" x="7.239" y="6.731" size="0.6096" layer="27" font="vector" ratio="15" rot="R180" align="center"/>
@@
 </element>
 <element name="L1" library="bschulz" package="0805" value="2.2uH" x="7.747" y="8.89" smashed="yes">
+<attribute name="DIGIKEY" value="732-2953-1-ND" x="7.747" y="8.89" size="1.778" layer="27" display="off"/>
+<attribute name="MF" value="Wurth" x="7.747" y="8.89" size="1.778" layer="27" display="off"/>
+<attribute name="MPN" value="74479775222" x="7.747" y="8.89" size="1.778" layer="27" display="off"/>
 <attribute name="NAME" x="5.715" y="8.89" size="0.6096" layer="25" font="vector" ratio="15" rot="R90" align="center"/>
 <attribute name="VALUE" x="7.747" y="7.493" size="0.6096" layer="27" font="vector" ratio="15" align="center"/>
@@
 <attribute name="VALUE" x="7.747" y="3.556" size="0.6096" layer="27" font="vector" ratio="15" rot="R90" align="center"/>
 </element>
-<element name="R2" library="bschulz_passives" package="R0402" value="" x="16.637" y="8.763" smashed="yes" rot="R180">
+<element name="R2" library="bschulz_passives" package="R0402" value="10k" x="16.637" y="8.763" smashed="yes" rot="R180">
 <attribute name="DIGIKEY" value="311-10.0KHRCT-ND" x="16.637" y="8.763" size="1.778" layer="27" rot="R180" display="off"/>
 <attribute name="MF" value="Yageo" x="16.637" y="8.763" size="1.778" layer="27" rot="R180" display="off"/>
@@
 <attribute name="VALUE_PART" value="10k" x="16.637" y="8.763" size="1.778" layer="27" rot="R180" display="off"/>
 </element>
-<element name="R3" library="bschulz_passives" package="R0402" value="" x="16.637" y="2.159" smashed="yes" rot="R180">
+<element name="R3" library="bschulz_passives" package="R0402" value="10k" x="16.637" y="2.159" smashed="yes" rot="R180">
 <attribute name="DIGIKEY" value="311-10.0KHRCT-ND" x="16.637" y="2.159" size="1.778" layer="27" rot="R180" display="off"/>
 <attribute name="MF" value="Yageo" x="16.637" y="2.159" size="1.778" layer="27" rot="R180" display="off"/>
